Commit message: Reordered project

File: ROS_Packages/allegro_hand_visual_control/allegro_hand_description/allegro_hand_description_right.urdf (robot description, URDF)
Before this commit: robot allegro_hand_right, 22 links, 21 joints
Links:
- link link_0.0: geometry collision box size=0.0196 0.0275 0.0164; visual mesh filename=package://allegro_hand_visual_control/allegro_hand_descript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
- link link_1.0: geometry collision box size=0.0196 0.0275 0.054; visual mesh filename=package://allegro_hand_visual_control/allegro_hand_descript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
- link link_10.0: geometry collision box size=0.0196 0.0275 0.0384; visual mesh filename=package://allegro_hand_visual_control/allegro_hand_descript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
- link link_11.0: geometry collision box size=0.0196 0.0275 0.0267; visual mesh filename=package://allegro_hand_visual_control/allegro_hand_descript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
- link link_11.0_tip: geometry collision sphere radius=0.012; visual mesh filename=package://allegro_hand_visual_control/allegro_hand_descript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
- link link_12.0: geometry collision box size=0.0358 0.034 0.0455; visual mesh filename=package://allegro_hand_visual_control/allegro_hand_descript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
- link link_13.0: geometry collision box size=0.0196 0.0275 0.0177; visual mesh filename=package://allegro_hand_visual_control/allegro_hand_descript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
- link link_14.0: geometry collision box size=0.0196 0.0275 0.0514; visual mesh filename=package://allegro_hand_visual_control/allegro_hand_descript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
- link link_15.0: geometry collision box size=0.0196 0.0275 0.0423; visual mesh filename=package://allegro_hand_visual_control/allegro_hand_descript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
- link link_15.0_tip: geometry collision sphere radius=0.012; visual mesh filename=package://allegro_hand_visual_control/allegro_hand_descript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
- link link_2.0: geometry collision box size=0.0196 0.0275 0.0384; visual mesh filename=package://allegro_hand_visual_control/allegro_hand_descript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
- link link_3.0: geometry collision box size=0.0196 0.0275 0.0267; visual mesh filename=package://allegro_hand_visual_control/allegro_hand_descript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
- link link_3.0_tip: geometry collision sphere radius=0.012; visual mesh filename=package://allegro_hand_visual_control/allegro_hand_descript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
- link link_4.0: geometry collision box size=0.0196 0.0275 0.0164; visual mesh filename=package://allegro_hand_visual_control/allegro_hand_descript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
- link link_5.0: geometry collision box size=0.0196 0.0275 0.054; visual mesh filename=package://allegro_hand_visual_control/allegro_hand_descript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
- link link_6.0: geometry collision box size=0.0196 0.0275 0.0384; visual mesh filename=package://allegro_hand_visual_control/allegro_hand_descript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
- link link_7.0: geometry collision box size=0.0196 0.0275 0.0267; visual mesh filename=package://allegro_hand_visual_control/allegro_hand_descript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
- link link_7.0_tip: geometry collision sphere radius=0.012; visual mesh filename=package://allegro_hand_visual_control/allegro_hand_descript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
- link link_8.0: geometry collision box size=0.0196 0.0275 0.0164; visual mesh filename=package://allegro_hand_visual_control/allegro_hand_descript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
- link link_9.0: geometry collision box size=0.0196 0.0275 0.054; visual mesh filename=package://allegro_hand_visual_control/allegro_hand_descript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
- link palm_link: geometry collision box size=0.0408 0.1130 0.095; visual mesh filename=package://allegro_hand_visual_control/allegro_hand_descript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
